Commit message: Fix link colors and joint limits.

File: urdf/mh24_macro.xacro (robot description, xacro)
@@ -2,4 +2,5 @@
 <robot xmlns:xacro="http://ros.org/wiki/xacro">
 	<xacro:macro name="motoman_mh24" params="prefix">
+		<xacro:property name="pi" value="3.14159265358979323846264338327950288419716" />
 		<!-- link list -->
 		<link name="${prefix}base_link">
@@ -61,5 +62,5 @@
 					<mesh filename="package://motoman_mh24_support/meshes/mh24/visual/u_axis.stl"/>
 				</geometry>
-				<material name="blue"/>
+				<material name="silver"/>
 			</visual>
 			<collision>
@@ -77,5 +78,5 @@
 					<mesh filename="package://motoman_mh24_support/meshes/mh24/visual/r_axis.stl"/>
 				</geometry>
-				<material name="silver"/>
+				<material name="blue"/>
 			</visual>
 			<collision>
@@ -93,5 +94,5 @@
 					<mesh filename="package://motoman_mh24_support/meshes/mh24/visual/b_axis.stl"/>
 				</geometry>
-				<material name="blue"/>
+				<material name="silver"/>
 			</visual>
 			<collision>
@@ -108,5 +109,5 @@
 					<mesh filename="package://motoman_mh24_support/meshes/mh24/visual/t_axis.stl" />
 				</geometry>
-				<material name="silver"/>
+				<material name="blue"/>
 			</visual>
 			<collision>
@@ -124,5 +125,5 @@
 			<origin xyz="0 0 0" rpy="0 0 0"/>
 			<axis xyz="0 0 1" />
-			<limit lower="-2.9671" upper="2.9671" effort="100" velocity="2.96" />
+			<limit lower="${-180 / 180.0 * pi}" upper="${180 / 180.0 * pi}" effort="100" velocity="3.44" />
 		</joint>
 		<joint name="${prefix}joint_l" type="revolute">
@@ -131,5 +132,5 @@
 			<origin xyz="0.150 0 0.505" rpy="0 0 0"/>
 			<axis xyz="0 1 0" />
-			<limit lower="-1.1345" upper="2.6180" effort="100" velocity="2.96" />
+			<limit lower="${-105 / 180.0 * pi}" upper="${155 / 180.0 * pi}" effort="100" velocity="3.32" />
 		</joint>
 		<joint name="${prefix}joint_u" type="revolute">
@@ -138,5 +139,6 @@
 			<origin xyz="0 0 0.760" rpy="0 0 0"/>
 			<axis xyz="0 -1 0" />
-			<limit lower="-1.0122" upper="3.2218" effort="100" velocity="2.96" />
+			<!-- Limited wrt to datasheet to prevent self-collisions -->
+			<limit lower="${-86 / 180.0 * pi}" upper="${163 / 180.0 * pi}" effort="100" velocity="3.67" />
 		</joint>
 		<joint name="${prefix}joint_r" type="revolute">
@@ -145,5 +147,5 @@
 			<origin xyz="0 0 0.200" rpy="0 0 0"/>
 			<axis xyz="-1 0 0" />
-			<limit lower="-3.3161" upper="3.3161" effort="100" velocity="3.48" />
+			<limit lower="${-200 / 180.0 * pi}" upper="${200 / 180.0 * pi}" effort="100" velocity="7.16" />
 		</joint>
 		<joint name="${prefix}joint_b" type="revolute">
@@ -152,5 +154,5 @@
 			<origin xyz="0.795 0 0" rpy="0 0 0"/>
 			<axis xyz="0 -1 0" />
-			<limit lower="-2.1817" upper="2.1817" effort="100" velocity="3.48" />
+			<limit lower="${-150 / 180.0 * pi}" upper="${150 / 180.0 * pi}" effort="100" velocity="7.16" />
 		</joint>
 		<joint name="${prefix}joint_t" type="revolute">
@@ -159,5 +161,5 @@
 			<origin xyz="0.100 0 0" rpy="0 0 0"/>
 			<axis xyz="-1 0 0" />
-			<limit lower="-6.2831" upper="6.2831" effort="100" velocity="6.97" />
+			<limit lower="${-455 / 180.0 * pi}" upper="${455 / 180.0 * pi}" effort="100" velocity="10.82" />
 		</joint>
 		<!-- end of joint list -->

Commit message: Add vendor frames.

File: urdf/mh24_macro.xacro (robot description, xacro)
@@ -24,4 +24,5 @@
 			</collision>
 		</link>
+		<link name="${prefix}vendor_base_link" />
 		<link name="${prefix}link_s">
 			<visual>
@@ -118,6 +119,12 @@
 			</collision>
 		</link>
+		<link name="${prefix}vendor_ee" />
 		<!-- end of link list -->
 		<!-- joint list -->
+		<joint name="${prefix}vendor_base_joint" type="fixed">
+			<parent link="${prefix}base_link" />
+			<child link="${prefix}vendor_base_link" />
+			<origin xyz="0 0 0.505" />
+		</joint>
 		<joint name="${prefix}joint_s" type="revolute">
 			<parent link="${prefix}base_link"/>
@@ -163,4 +170,9 @@
 			<limit lower="${-455 / 180.0 * pi}" upper="${455 / 180.0 * pi}" effort="100" velocity="10.82" />
 		</joint>
+		<joint name="${prefix}vendor_ee_joint" type="fixed">
+			<parent link="${prefix}link_t" />
+			<child link="${prefix}vendor_ee" />
+			<origin rpy="0 ${-0.5 * pi} ${pi}" />
+		</joint>
 		<!-- end of joint list -->
 	</xacro:macro>

Commit message: Remove wrong base mesh rotation.

File: urdf/mh24_macro.xacro (robot description, xacro)
@@ -6,5 +6,4 @@
 		<link name="${prefix}base_link">
 			<visual>
-			        <origin rpy="0 0 3.14159"/>
 				<geometry>
 					<mesh filename="package://yaskawa_mh24_support/meshes/mh24/visual/base_axis.stl" />
@@ -15,5 +14,4 @@
 			</visual>
 			<collision>
-			        <origin rpy="0 0 3.14159"/>
 				<geometry>
 					<mesh filename="package://yaskawa_mh24_support/meshes/mh24/collision/base_axis.stl" />
@@ -43,5 +41,4 @@
 		<link name="${prefix}link_l">
 			<visual>
-				<!-- <origin rpy="1.57 3.1416 0" xyz="0 0 0"/> -->
 				<geometry>
 					<mesh filename="package://yaskawa_mh24_support/meshes/mh24/visual/l_axis.stl"/>
@@ -50,5 +47,4 @@
 			</visual>
 			<collision>
-				<!-- <origin rpy="1.57 3.1416 0" xyz="0 0 0"/> -->
 				<geometry>
 					<mesh filename="package://yaskawa_mh24_support/meshes/mh24/collision/l_axis.stl" />
@@ -59,5 +55,4 @@
 		<link name="${prefix}link_u">
 			<visual>
-				<!-- <origin rpy="1.57 -3.1415 0" xyz="0 0 0"/> -->
 				<geometry>
 					<mesh filename="package://yaskawa_mh24_support/meshes/mh24/visual/u_axis.stl"/>
@@ -66,5 +61,4 @@
 			</visual>
 			<collision>
-				<!-- <origin rpy="1.57 -3.1415 0" xyz="0 0 0"/> -->
 				<geometry>
 					<mesh filename="package://yaskawa_mh24_support/meshes/mh24/collision/u_axis.stl" />
@@ -75,5 +69,4 @@
 		<link name="${prefix}link_r">
 			<visual>
-				<!-- <origin rpy="0 0 3.1416" xyz="0 0 0"/> -->
 				<geometry>
 					<mesh filename="package://yaskawa_mh24_support/meshes/mh24/visual/r_axis.stl"/>
@@ -82,5 +75,4 @@
 			</visual>
 			<collision>
-				<!-- <origin rpy="0 0 3.1416" xyz="0 0 0"/> -->
 				<geometry>
 					<mesh filename="package://yaskawa_mh24_support/meshes/mh24/collision/r_axis.stl" />
@@ -91,5 +83,4 @@
 		<link name="${prefix}link_b">
 			<visual>
-				<!-- <origin rpy="-1.57 0 3.1416" xyz="0 0 0"/> -->
 				<geometry>
 					<mesh filename="package://yaskawa_mh24_support/meshes/mh24/visual/b_axis.stl"/>
@@ -98,5 +89,4 @@
 			</visual>
 			<collision>
-				<!-- <origin rpy="-1.57 0 3.1416" xyz="0 0 0"/> -->
 				<geometry>
 					<mesh filename="package://yaskawa_mh24_support/meshes/mh24/collision/b_axis.stl" />
