Commit message: Rename to yaskawa_mh24_support

File: urdf/mh24.xacro (robot description, xacro)
@@ -1,5 +1,5 @@
 <?xml version="1.0" ?>
-<robot name="motoman_mh24" xmlns:xacro="http://ros.org/wiki/xacro">
-	<xacro:include filename="$(find motoman_mh24_support)/urdf/mh24_macro.xacro" />
-	<xacro:motoman_mh24 prefix=""/>
+<robot name="yaskawa_mh24" xmlns:xacro="http://ros.org/wiki/xacro">
+	<xacro:include filename="$(find yaskawa_mh24_support)/urdf/mh24_macro.xacro" />
+	<xacro:yaskawa_mh24 prefix=""/>
 </robot>

File: urdf/mh24_macro.xacro (robot description, xacro)
@@ -1,5 +1,5 @@
 <?xml version="1.0" ?>
 <robot xmlns:xacro="http://ros.org/wiki/xacro">
-	<xacro:macro name="motoman_mh24" params="prefix">
+	<xacro:macro name="yaskawa_mh24" params="prefix">
 		<xacro:property name="pi" value="3.14159265358979323846264338327950288419716" />
 		<!-- link list -->
@@ -8,5 +8,5 @@
 			        <origin rpy="0 0 3.14159"/>
 				<geometry>
-					<mesh filename="package://motoman_mh24_support/meshes/mh24/visual/base_axis.stl" />
+					<mesh filename="package://yaskawa_mh24_support/meshes/mh24/visual/base_axis.stl" />
 				</geometry>
 				<material name="blue">
@@ -17,5 +17,5 @@
 			        <origin rpy="0 0 3.14159"/>
 				<geometry>
-					<mesh filename="package://motoman_mh24_support/meshes/mh24/collision/base_axis.stl" />
+					<mesh filename="package://yaskawa_mh24_support/meshes/mh24/collision/base_axis.stl" />
 				</geometry>
 				<material name="yellow">
@@ -27,5 +27,5 @@
 			<visual>
 				<geometry>
-					<mesh filename="package://motoman_mh24_support/meshes/mh24/visual/s_axis.stl"/>
+					<mesh filename="package://yaskawa_mh24_support/meshes/mh24/visual/s_axis.stl"/>
 				</geometry>
 				<material name="silver">
@@ -35,5 +35,5 @@
 			<collision>
 				<geometry>
-					<mesh filename="package://motoman_mh24_support/meshes/mh24/collision/s_axis.stl" />
+					<mesh filename="package://yaskawa_mh24_support/meshes/mh24/collision/s_axis.stl" />
 				</geometry>
 				<material name="yellow"/>
@@ -44,5 +44,5 @@
 				<!-- <origin rpy="1.57 3.1416 0" xyz="0 0 0"/> -->
 				<geometry>
-					<mesh filename="package://motoman_mh24_support/meshes/mh24/visual/l_axis.stl"/>
+					<mesh filename="package://yaskawa_mh24_support/meshes/mh24/visual/l_axis.stl"/>
 				</geometry>
 				<material name="blue"/>
@@ -51,5 +51,5 @@
 				<!-- <origin rpy="1.57 3.1416 0" xyz="0 0 0"/> -->
 				<geometry>
-					<mesh filename="package://motoman_mh24_support/meshes/mh24/collision/l_axis.stl" />
+					<mesh filename="package://yaskawa_mh24_support/meshes/mh24/collision/l_axis.stl" />
 				</geometry>
 				<material name="yellow"/>
@@ -60,5 +60,5 @@
 				<!-- <origin rpy="1.57 -3.1415 0" xyz="0 0 0"/> -->
 				<geometry>
-					<mesh filename="package://motoman_mh24_support/meshes/mh24/visual/u_axis.stl"/>
+					<mesh filename="package://yaskawa_mh24_support/meshes/mh24/visual/u_axis.stl"/>
 				</geometry>
 				<material name="silver"/>
@@ -67,5 +67,5 @@
 				<!-- <origin rpy="1.57 -3.1415 0" xyz="0 0 0"/> -->
 				<geometry>
-					<mesh filename="package://motoman_mh24_support/meshes/mh24/collision/u_axis.stl" />
+					<mesh filename="package://yaskawa_mh24_support/meshes/mh24/collision/u_axis.stl" />
 				</geometry>
 				<material name="yellow"/>
@@ -76,5 +76,5 @@
 				<!-- <origin rpy="0 0 3.1416" xyz="0 0 0"/> -->
 				<geometry>
-					<mesh filename="package://motoman_mh24_support/meshes/mh24/visual/r_axis.stl"/>
+					<mesh filename="package://yaskawa_mh24_support/meshes/mh24/visual/r_axis.stl"/>
 				</geometry>
 				<material name="blue"/>
@@ -83,5 +83,5 @@
 				<!-- <origin rpy="0 0 3.1416" xyz="0 0 0"/> -->
 				<geometry>
-					<mesh filename="package://motoman_mh24_support/meshes/mh24/collision/r_axis.stl" />
+					<mesh filename="package://yaskawa_mh24_support/meshes/mh24/collision/r_axis.stl" />
 				</geometry>
 				<material name="yellow"/>
@@ -92,5 +92,5 @@
 				<!-- <origin rpy="-1.57 0 3.1416" xyz="0 0 0"/> -->
 				<geometry>
-					<mesh filename="package://motoman_mh24_support/meshes/mh24/visual/b_axis.stl"/>
+					<mesh filename="package://yaskawa_mh24_support/meshes/mh24/visual/b_axis.stl"/>
 				</geometry>
 				<material name="silver"/>
@@ -99,5 +99,5 @@
 				<!-- <origin rpy="-1.57 0 3.1416" xyz="0 0 0"/> -->
 				<geometry>
-					<mesh filename="package://motoman_mh24_support/meshes/mh24/collision/b_axis.stl" />
+					<mesh filename="package://yaskawa_mh24_support/meshes/mh24/collision/b_axis.stl" />
 				</geometry>
 				<material name="yellow"/>
@@ -107,5 +107,5 @@
 			<visual>
 				<geometry>
-					<mesh filename="package://motoman_mh24_support/meshes/mh24/visual/t_axis.stl" />
+					<mesh filename="package://yaskawa_mh24_support/meshes/mh24/visual/t_axis.stl" />
 				</geometry>
 				<material name="blue"/>
@@ -113,5 +113,5 @@
 			<collision>
 				<geometry>
-					<mesh filename="package://motoman_mh24_support/meshes/mh24/collision/t_axis.stl" />
+					<mesh filename="package://yaskawa_mh24_support/meshes/mh24/collision/t_axis.stl" />
 				</geometry>
 				<material name="yellow"/>

Commit message: Rename meshes, use Collada smooth meshes for visual, add test file, fix interface streaming file name, improve XACRO definition

File: urdf/mh24.xacro (robot description, xacro)
@@ -1,5 +1,5 @@
 <?xml version="1.0" ?>
-<robot name="yaskawa_mh24" xmlns:xacro="http://ros.org/wiki/xacro">
-	<xacro:include filename="$(find yaskawa_mh24_support)/urdf/mh24_macro.xacro" />
-	<xacro:yaskawa_mh24 prefix=""/>
+<robot name="motoman_mh_24" xmlns:xacro="http://ros.org/wiki/xacro">
+  <xacro:include filename="$(find yaskawa_mh24_support)/urdf/mh24_macro.xacro"/>
+  <xacro:motoman_mh_24 prefix=""/>
 </robot>

File: urdf/mh24_macro.xacro (robot description, xacro)
@@ -1,169 +1,181 @@
 <?xml version="1.0" ?>
 <robot xmlns:xacro="http://ros.org/wiki/xacro">
-	<xacro:macro name="yaskawa_mh24" params="prefix">
-		<xacro:property name="pi" value="3.14159265358979323846264338327950288419716" />
-		<!-- link list -->
-		<link name="${prefix}base_link">
-			<visual>
-				<geometry>
-					<mesh filename="package://yaskawa_mh24_support/meshes/mh24/visual/base_axis.stl" />
-				</geometry>
-				<material name="blue">
-					<color rgba="0 0 1 1"/>
-				</material>
-			</visual>
-			<collision>
-				<geometry>
-					<mesh filename="package://yaskawa_mh24_support/meshes/mh24/collision/base_axis.stl" />
-				</geometry>
-				<material name="yellow">
-					<color rgba="0 1 1 1"/>
-				</material>
-			</collision>
-		</link>
-		<link name="${prefix}vendor_base_link" />
-		<link name="${prefix}link_s">
-			<visual>
-				<geometry>
-					<mesh filename="package://yaskawa_mh24_support/meshes/mh24/visual/s_axis.stl"/>
-				</geometry>
-				<material name="silver">
-					<color rgba="0.8 0.8 0.8 1"/>
-				</material>
-			</visual>
-			<collision>
-				<geometry>
-					<mesh filename="package://yaskawa_mh24_support/meshes/mh24/collision/s_axis.stl" />
-				</geometry>
-				<material name="yellow"/>
-			</collision>
-		</link>
-		<link name="${prefix}link_l">
-			<visual>
-				<geometry>
-					<mesh filename="package://yaskawa_mh24_support/meshes/mh24/visual/l_axis.stl"/>
-				</geometry>
-				<material name="blue"/>
-			</visual>
-			<collision>
-				<geometry>
-					<mesh filename="package://yaskawa_mh24_support/meshes/mh24/collision/l_axis.stl" />
-				</geometry>
-				<material name="yellow"/>
-			</collision>
-		</link>
-		<link name="${prefix}link_u">
-			<visual>
-				<geometry>
-					<mesh filename="package://yaskawa_mh24_support/meshes/mh24/visual/u_axis.stl"/>
-				</geometry>
-				<material name="silver"/>
-			</visual>
-			<collision>
-				<geometry>
-					<mesh filename="package://yaskawa_mh24_support/meshes/mh24/collision/u_axis.stl" />
-				</geometry>
-				<material name="yellow"/>
-			</collision>
-		</link>
-		<link name="${prefix}link_r">
-			<visual>
-				<geometry>
-					<mesh filename="package://yaskawa_mh24_support/meshes/mh24/visual/r_axis.stl"/>
-				</geometry>
-				<material name="blue"/>
-			</visual>
-			<collision>
-				<geometry>
-					<mesh filename="package://yaskawa_mh24_support/meshes/mh24/collision/r_axis.stl" />
-				</geometry>
-				<material name="yellow"/>
-			</collision>
-		</link>
-		<link name="${prefix}link_b">
-			<visual>
-				<geometry>
-					<mesh filename="package://yaskawa_mh24_support/meshes/mh24/visual/b_axis.stl"/>
-				</geometry>
-				<material name="silver"/>
-			</visual>
-			<collision>
-				<geometry>
-					<mesh filename="package://yaskawa_mh24_support/meshes/mh24/collision/b_axis.stl" />
-				</geometry>
-				<material name="yellow"/>
-			</collision>
-		</link>
-		<link name="${prefix}link_t">
-			<visual>
-				<geometry>
-					<mesh filename="package://yaskawa_mh24_support/meshes/mh24/visual/t_axis.stl" />
-				</geometry>
-				<material name="blue"/>
-			</visual>
-			<collision>
-				<geometry>
-					<mesh filename="package://yaskawa_mh24_support/meshes/mh24/collision/t_axis.stl" />
-				</geometry>
-				<material name="yellow"/>
-			</collision>
-		</link>
-		<link name="${prefix}vendor_ee" />
-		<!-- end of link list -->
-		<!-- joint list -->
-		<joint name="${prefix}vendor_base_joint" type="fixed">
-			<parent link="${prefix}base_link" />
-			<child link="${prefix}vendor_base_link" />
-			<origin xyz="0 0 0.505" />
-		</joint>
-		<joint name="${prefix}joint_s" type="revolute">
-			<parent link="${prefix}base_link"/>
-			<child link="${prefix}link_s"/>
-			<origin xyz="0 0 0" />
-			<axis xyz="0 0 1" />
-			<limit lower="${-180 / 180.0 * pi}" upper="${180 / 180.0 * pi}" effort="100" velocity="3.44" />
-		</joint>
-		<joint name="${prefix}joint_l" type="revolute">
-			<parent link="${prefix}link_s"/>
-			<child link="${prefix}link_l"/>
-			<origin xyz="0.150 0 0.505" />
-			<axis xyz="0 1 0" />
-			<limit lower="${-105 / 180.0 * pi}" upper="${155 / 180.0 * pi}" effort="100" velocity="3.32" />
-		</joint>
-		<joint name="${prefix}joint_u" type="revolute">
-			<parent link="${prefix}link_l"/>
-			<child link="${prefix}link_u"/>
-			<origin xyz="0 0 0.760" />
-			<axis xyz="0 -1 0" />
-			<!-- Limited wrt to datasheet to prevent self-collisions -->
-			<limit lower="${-86 / 180.0 * pi}" upper="${163 / 180.0 * pi}" effort="100" velocity="3.67" />
-		</joint>
-		<joint name="${prefix}joint_r" type="revolute">
-			<parent link="${prefix}link_u"/>
-			<child link="${prefix}link_r"/>
-			<origin xyz="0 0 0.200" />
-			<axis xyz="-1 0 0" />
-			<limit lower="${-200 / 180.0 * pi}" upper="${200 / 180.0 * pi}" effort="100" velocity="7.16" />
-		</joint>
-		<joint name="${prefix}joint_b" type="revolute">
-			<parent link="${prefix}link_r"/>
-			<child link="${prefix}link_b"/>
-			<origin xyz="0.795 0 0" />
-			<axis xyz="0 -1 0" />
-			<limit lower="${-150 / 180.0 * pi}" upper="${150 / 180.0 * pi}" effort="100" velocity="7.16" />
-		</joint>
-		<joint name="${prefix}joint_t" type="revolute">
-			<parent link="${prefix}link_b"/>
-			<child link="${prefix}link_t"/>
-			<origin xyz="0.100 0 0" />
-			<axis xyz="-1 0 0" />
-			<limit lower="${-455 / 180.0 * pi}" upper="${455 / 180.0 * pi}" effort="100" velocity="10.82" />
-		</joint>
-		<joint name="${prefix}vendor_ee_joint" type="fixed">
-			<parent link="${prefix}link_t" />
-			<child link="${prefix}vendor_ee" />
-			<origin rpy="0 ${-0.5 * pi} ${pi}" />
-		</joint>
-		<!-- end of joint list -->
-	</xacro:macro>
+  <xacro:macro name="motoman_mh_24" params="prefix">
+    <!-- link list -->
+    <link name="${prefix}base_link">
+      <visual>
+        <origin xyz="0 0 0" rpy="0 0 0"/>
+        <geometry>
+          <mesh filename="package://yaskawa_mh24_support/meshes/mh24/visual/base_link.dae"/>
+        </geometry>
+        <material name="blue">
+          <color rgba="0 0 1 1"/>
+        </material>
+      </visual>
+      <collision>
+        <origin xyz="0 0 0" rpy="0 0 0"/>
+        <geometry>
+          <mesh filename="package://yaskawa_mh24_support/meshes/mh24/collision/base_link.stl"/>
+        </geometry>
+        <material name="blue">
+          <color rgba="0 0 1 1"/>
+        </material>
+      </collision>
+    </link>
+    <link name="${prefix}link_s">
+      <visual>
+        <origin xyz="0 0 0" rpy="0 0 0"/>
+        <geometry>
+          <mesh filename="package://yaskawa_mh24_support/meshes/mh24/visual/link_s.dae"/>
+        </geometry>
+        <material name="blue"/>
+      </visual>
+      <collision>
+        <origin xyz="0 0 0" rpy="0 0 0"/>
+        <geometry>
+          <mesh filename="package://yaskawa_mh24_support/meshes/mh24/collision/link_s.stl"/>
+        </geometry>
+        <material name="blue"/>
+      </collision>
+    </link>
+    <link name="${prefix}link_l">
+      <visual>
+        <origin xyz="0 0 0" rpy="0 0 0"/>
+        <geometry>
+          <mesh filename="package://yaskawa_mh24_support/meshes/mh24/visual/link_l.dae"/>
+        </geometry>
+        <material name="blue"/>
+      </visual>
+      <collision>
+        <origin xyz="0 0 0" rpy="0 0 0"/>
+        <geometry>
+          <mesh filename="package://yaskawa_mh24_support/meshes/mh24/collision/link_l.stl"/>
+        </geometry>
+        <material name="blue"/>
+      </collision>
+    </link>
+    <link name="${prefix}link_u">
+      <visual>
+        <origin xyz="0 0 0" rpy="0 0 0"/>
+        <geometry>
+          <mesh filename="package://yaskawa_mh24_support/meshes/mh24/visual/link_u.dae"/>
+        </geometry>
+        <material name="blue"/>
+      </visual>
+      <collision>
+        <origin xyz="0 0 0" rpy="0 0 0"/>
+        <geometry>
+          <mesh filename="package://yaskawa_mh24_support/meshes/mh24/collision/link_u.stl"/>
+        </geometry>
+        <material name="blue"/>
+      </collision>
+    </link>
+    <link name="${prefix}link_r">
+      <visual>
+        <origin xyz="0 0 0" rpy="0 0 0"/>
+        <geometry>
+          <mesh filename="package://yaskawa_mh24_support/meshes/mh24/visual/link_r.dae"/>
+        </geometry>
+        <material name="blue"/>
+      </visual>
+      <collision>
+        <origin xyz="0 0 0" rpy="0 0 0"/>
+        <geometry>
+          <mesh filename="package://yaskawa_mh24_support/meshes/mh24/collision/link_r.stl"/>
+        </geometry>
+        <material name="blue"/>
+      </collision>
+    </link>
+    <link name="${prefix}link_b">
+      <visual>
+        <origin xyz="0 0 0" rpy="0 0 0"/>
+        <geometry>
+          <mesh filename="package://yaskawa_mh24_support/meshes/mh24/visual/link_b.dae"/>
+        </geometry>
+        <material name="blue"/>
+      </visual>
+      <collision>
+        <origin xyz="0 0 0" rpy="0 0 0"/>
+        <geometry>
+          <mesh filename="package://yaskawa_mh24_support/meshes/mh24/collision/link_b.stl"/>
+        </geometry>
+        <material name="blue"/>
+      </collision>
+    </link>
+    <link name="${prefix}link_t">
+      <visual>
+        <origin xyz="0 0 0" rpy="0 0 0"/>
+        <geometry>
+          <mesh filename="package://yaskawa_mh24_support/meshes/mh24/visual/link_t.dae"/>
+        </geometry>
+        <material name="blue"/>
+      </visual>
+      <collision>
+        <origin xyz="0 0 0" rpy="0 0 0"/>
+        <geometry>
+          <mesh filename="package://yaskawa_mh24_support/meshes/mh24/collision/link_t.stl"/>
+        </geometry>
+        <material name="blue"/>
+      </collision>
+    </link>
+    <link name="${prefix}tool0"/>
+    <!-- end of link list -->
+    <!-- joint list -->
+    <joint name="${prefix}joint_s" type="revolute">
+      <origin xyz="0 0 0" rpy="0 0 0"/>
+      <parent link="${prefix}base_link"/>
+      <child link="${prefix}link_s"/>
+      <axis xyz="0 0 1"/>
+      <limit lower="${-180 / 180.0 * pi}" upper="${180 / 180.0 * pi}" effort="0" velocity="${radians(197)}"/>
+    </joint>
+    <joint name="${prefix}joint_l" type="revolute">
+      <origin xyz="0.150 0 0.505" rpy="0 0 0"/>
+      <parent link="${prefix}link_s"/>
+      <child link="${prefix}link_l"/>
+      <axis xyz="0 1 0"/>
+      <limit lower="${-105 / 180.0 * pi}" upper="${155 / 180.0 * pi}" effort="0" velocity="${radians(190)}"/>
+    </joint>
+    <joint name="${prefix}joint_u" type="revolute">
+      <origin xyz="0 0 0.760" rpy="0 0 0"/>
+      <parent link="${prefix}link_l"/>
+      <child link="${prefix}link_u"/>
+      <axis xyz="0 -1 0"/>
+      <!-- Limited wrt to datasheet to prevent self-collisions -->
+      <limit lower="${-86 / 180.0 * pi}" upper="${163 / 180.0 * pi}" effort="0" velocity="${radians(210)}"/>
+    </joint>
+    <joint name="${prefix}joint_r" type="revolute">
+      <origin xyz="0 0 0.200" rpy="0 0 0"/>
+      <parent link="${prefix}link_u"/>
+      <child link="${prefix}link_r"/>
+      <axis xyz="-1 0 0"/>
+      <limit lower="${-200 / 180.0 * pi}" upper="${200 / 180.0 * pi}" effort="0" velocity="${radians(410)}"/>
+    </joint>
+    <joint name="${prefix}joint_b" type="revolute">
+      <origin xyz="0.795 0 0" rpy="0 0 0"/>
+      <parent link="${prefix}link_r"/>
+      <child link="${prefix}link_b"/>
+      <axis xyz="0 -1 0"/>
+      <limit lower="${-150 / 180.0 * pi}" upper="${150 / 180.0 * pi}" effort="0" velocity="${radians(410)}"/>
+    </joint>
+    <joint name="${prefix}joint_t" type="revolute">
+      <origin xyz="0.100 0 0" rpy="0 0 0"/>
+      <parent link="${prefix}link_b"/>
+      <child link="${prefix}link_t"/>
+      <axis xyz="-1 0 0"/>
+      <limit lower="${-455 / 180.0 * pi}" upper="${455 / 180.0 * pi}" effort="0" velocity="${radians(620)}"/>
+    </joint>
+    <joint name="${prefix}joint_t-tool0" type="fixed">
+      <origin xyz="0 0 0" rpy="0 ${-0.5 * pi} ${pi}"/>
+      <parent link="${prefix}link_t"/>
+      <child link="${prefix}tool0"/>
+    </joint>
+    <!-- end of joint list -->
+    <!-- ROS base_link to Robot Manufacturer World Coordinates transform -->
+    <link name="${prefix}base"/>
+    <joint name="${prefix}base_link-base" type="fixed">
+      <origin xyz="0 0 0.505" rpy="0 0 0"/>
+      <parent link="${prefix}base_link"/>
+      <child link="${prefix}base"/>
+    </joint>
+  </xacro:macro>
 </robot>
